File: sensor_sigfox_1.1/_autosave-sensor_sigfox_1.1.kicad_sch (KiCad schematic)
At the start: 18 parts, among them IC1 WSSFM11R2DAT, J1 Battery, J2 Conn_01x07_Socket, J3 Conn_01x01_Female, J4 Antenna, U1 ATtiny826-X, U2 MLX90393, Y1 32.768 kHz

Commit message: revision 1.1.1
Parts:
- removed J4: Antenna, Connector_Coaxial:U.FL_Hirose_U.FL-R-SMT-1_Vertical, symbol Connector:Conn_Coaxial
Connections:
- net GND: now also U2.4 (N/C)
Changed lines of the file:
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@@
   (junction (at 102.87 123.19) (diameter 0) (color 0 0 0 0)
   )
+  (junction (at 156.21 133.35) (diameter 0) (color 0 0 0 0)
+  )
   (junction (at 125.73 104.14) (diameter 0) (color 0 0 0 0)
   )
@@
     (stroke (width 0) (type default))
   )
+  (wire (pts (xy 166.37 119.38) (xy 166.37 133.35))
+    (stroke (width 0) (type default))
+  )
   (wire (pts (xy 142.24 45.72) (xy 224.79 45.72))
     (stroke (width 0) (type default))
@@
     (stroke (width 0) (type default))
   )
+  (wire (pts (xy 166.37 133.35) (xy 156.21 133.35))
+    (stroke (width 0) (type default))
+  )
   (wire (pts (xy 125.73 104.14) (xy 125.73 101.6))
     (stroke (width 0) (type default))
@@
   )
   (wire (pts (xy 110.49 83.82) (xy 110.49 86.36))
+    (stroke (width 0) (type default))
+  )
+  (wire (pts (xy 162.56 119.38) (xy 166.37 119.38))
     (stroke (width 0) (type default))
   )
@@
         )
       )
-    )
-  )
-  (symbol (lib_id "Connector:Conn_Coaxial") (at 231.14 86.36 0) (unit 1)
-    (in_bom yes) (on_board yes) (dnp no) (fields_autoplaced)
-    (property "Reference" "J4" (at 233.68 85.3831 0)
-      (effects (font (size 1.27 1.27)) (justify left))
-    )
-    (property "Value" "Antenna" (at 233.68 87.9231 0)
-      (effects (font (size 1.27 1.27)) (justify left))
-    )
-    (property "Footprint" "Connector_Coaxial:U.FL_Hirose_U.FL-R-SMT-1_Vertical" (at 231.14 86.36 0)
-      (effects (font (size 1.27 1.27)) hide)
-    )
-    (property "Datasheet" " ~" (at 231.14 86.36 0)
-      (effects (font (size 1.27 1.27)) hide)
-    )
-    (pin "1")
-    (pin "2")
-    (instances
-      (project "sensor_sigfox_1.1"
-        (path "/7e4087c3-8cfe-4a56-93d2-ee627c3b6019"
-          (reference "J4") (unit 1)
-        )
-      )
